Commit message: combine phobos and phobos_nuclear into one package

File: urdf/phobos.urdf.xacro (robot description, xacro)
@@ -1,55 +1,127 @@
 <?xml version="1.0"?>
 <!--
-Copyright (c) 2018, I3D Robotics Ltd.
+Copyright (c) 2019, I3D Robotics Ltd.
 -->
 <robot xmlns:xacro="http://ros.org/wiki/xacro">
-    <xacro:macro name="phobos_camera">
-    <link name="cameraLeft_optical" />
-    <link name="cameraRight_optical" />
-    <link name="cameraLeft" />
-    <link name="cameraRight" />
-    <link name="phobos_center">
-        <visual>
-            <!--<origin xyz="0.025 0 0.07" rpy="0 0 0"/>-->
-            <origin xyz="0.07 0 0.025" rpy="0 0 0"/>
-            <geometry>
-                <box size="0.140 0.390 0.05"/>
-                <!--mesh filename="package://deimos/urdf/phobos.stl" /-->
-            </geometry>
-            <material name="Orange">
-                <color rgba="1 0.5 0 1"/>
-            </material>
-        </visual>
-    </link>
-    <link name="phobos_depth_camera" />
-    <joint name="phobos_right_camera_joint" type="fixed">
-        <parent link="phobos_center"/>
-        <child link="cameraRight"/>
-        <!--<origin xyz="0.0245 0.148794 0.086874" rpy="0 0 0" />-->
-        <origin xyz="0.086874 -0.148794  0.0245" rpy="0 0 0" />
-    </joint>
-    <joint name="phobos_left_camera_joint" type="fixed">
-        <parent link="phobos_center"/>
-        <child link="cameraLeft"/>
-        <!--<origin xyz="0.0245 -0.148794 0.086874" rpy="0 0 0" />-->
-        <origin xyz="0.086874 0.148794 0.0245" rpy="0 0 0" />
-    </joint>
-    <joint name="phobos_left_optical_joint" type="fixed">
-        <parent link="cameraLeft"/>
-        <child link="cameraLeft_optical"/>
-	<!-- Correct for the optical frame orientation -->
-        <origin xyz="0 0 0" rpy="${-pi/2} 0 ${-pi/2}" />
-    </joint>
-    <joint name="phobos_right_optical_joint" type="fixed">
-        <parent link="cameraRight"/>
-        <child link="cameraRight_optical"/>
-	<!-- Correct for the optical frame orientation -->
-        <origin xyz="0 0 0" rpy="${-pi/2} 0 ${-pi/2}" />
-    </joint>
-    <joint name="phobos_depth_camera_joint" type="fixed">
-        <parent link="cameraLeft"/>
-        <child link="phobos_depth_camera"/>
-        <origin xyz="0 0 0" rpy="0 0 0" />
-    </joint>
+    <xacro:macro name="i3dr_phobos" params="camera_name:=phobos en_mesh:=true en_imu:=false">
+        <xacro:property name="height" value="0.05"/>
+        <xacro:property name="width" value="0.39"/>
+        <xacro:property name="length" value="0.14"/>
+        <!-- TODO reduce mesh resolution for faster loading -->
+        <xacro:property name="mesh_file" value="package://i3dr_phobos/mesh/phobos.stl"/>
+        <xacro:property name="mesh_offset_xyz" value="-0.07 0 0"/>
+        <xacro:property name="mesh_offset_rpy" value="0 ${pi} ${-pi/2}"/>
+        <xacro:property name="box_offset_xyz" value="0 0 ${height/2}"/>
+        <xacro:property name="box_offset_rpy" value="0 0 0"/>
+        <xacro:property name="toe_in_l" value="8.5"/>
+        <xacro:property name="toe_in_r" value="8.5"/>
+        <link name="${camera_name}_cameraLeft_optical" />
+        <link name="${camera_name}_cameraRight_optical" />
+        <link name="${camera_name}_cameraLeft" />
+        <link name="${camera_name}_cameraRight" />
+        <link name="${camera_name}_depth_optical_frame" />
+        <link name="${camera_name}_base_link" />
+        <link name="${camera_name}_mount_base_link" />
+        <xacro:if value="${(en_imu == 'true')}">
+            <link name="${camera_name}_imu_link"/>
+        </xacro:if>
+        <link name="${camera_name}_mount_point_1"/>
+        <link name="${camera_name}_mount_point_2"/>
+        <link name="${camera_name}_mount_point_3"/>
+        <link name="${camera_name}_mount_point_4"/>
+        <link name="${camera_name}_center">
+            <visual>
+                <xacro:if value="${(en_mesh == 'true')}">
+                    <origin xyz="${mesh_offset_xyz}" rpy="${mesh_offset_rpy}"/>
+                </xacro:if>
+                <xacro:if value="${(en_mesh == 'false')}">
+                    <origin xyz="${box_offset_xyz}" rpy="${box_offset_rpy}"/>
+                </xacro:if>
+                <geometry>
+                    <xacro:if value="${(en_mesh == 'true')}">
+                        <mesh filename="${mesh_file}"/>
+                    </xacro:if>
+                    <xacro:if value="${(en_mesh == 'false')}">
+                        <box size="${length} ${width} ${height}"/>
+                    </xacro:if>
+                </geometry>
+                <xacro:if value="${(en_mesh == 'false')}">
+                    <material name="${camera_name}_camera_colour">
+                        <color rgba="1 0.5 0.1 1"/>
+                    </material>
+                </xacro:if>
+            </visual>
+        </link>
+        <xacro:if value="${(en_imu == 'true')}">
+            <joint name="${camera_name}_imu_joint" type="fixed">
+                <origin xyz="0 0 0" rpy="0 0 ${pi}" />
+                <parent link="${camera_name}_base_link" />
+                <child link="${camera_name}_imu_link" />
+            </joint>
+            <joint name="${camera_name}_imu_mount_joint" type="fixed">
+                <origin xyz="0 0 0" rpy="0 0 ${pi}" />
+                <parent link="${camera_name}_base_link" />
+                <child link="${camera_name}_mount_base_link" />
+            </joint>
+        </xacro:if>
+        <xacro:if value="${(en_imu == 'false')}">
+            <joint name="${camera_name}_imu_mount_joint" type="fixed">
+                <origin xyz="0 0 0" rpy="0 0 0" />
+                <parent link="${camera_name}_base_link" />
+                <child link="${camera_name}_mount_base_link" />
+            </joint>
+        </xacro:if>
+        <joint name="${camera_name}_right_camera_joint" type="fixed">
+            <parent link="${camera_name}_center"/>
+            <child link="${camera_name}_cameraRight"/>
+            <origin xyz="${0.086874/2} ${-0.148794}  ${0.0245}" rpy="0 0 0" />
+        </joint>
+        <joint name="${camera_name}_left_camera_joint" type="fixed">
+            <parent link="${camera_name}_center"/>
+            <child link="${camera_name}_cameraLeft"/>
+            <origin xyz="${0.086874/2} ${0.148794}  ${0.0245}" rpy="0 0 0" />
+        </joint>
+        <joint name="${camera_name}_left_optical_joint" type="fixed">
+            <parent link="${camera_name}_cameraLeft"/>
+            <child link="${camera_name}_cameraLeft_optical"/>
+            <!-- Correct for the optical frame orientation -->
+            <origin xyz="0 0 0" rpy="${-pi/2} 0 ${(-pi/2)-(toe_in_l * (pi/180))}" />
+        </joint>
+        <joint name="${camera_name}_right_optical_joint" type="fixed">
+            <parent link="${camera_name}_cameraRight"/>
+            <child link="${camera_name}_cameraRight_optical"/>
+            <!-- Correct for the optical frame orientation -->
+            <origin xyz="0 0 0" rpy="${-pi/2} 0 ${(-pi/2)+(toe_in_r * (pi/180))}" />
+        </joint>
+        <joint name="${camera_name}_depth_optical_joint" type="fixed">
+            <parent link="${camera_name}_cameraLeft"/>
+            <child link="${camera_name}_depth_optical_frame"/>
+            <origin xyz="0 0 0" rpy="${-pi/2} 0 ${(-pi/2)}" />
+        </joint>
+        <joint name="${camera_name}_mount_center_joint" type="fixed">
+            <parent link="${camera_name}_mount_base_link"/>
+            <child link="${camera_name}_center"/>
+            <origin xyz="0 0 0" rpy="0 0 ${-pi/2}" />
+        </joint>
+        <joint name="${camera_name}_mount_point_1_joint" type="fixed">
+            <parent link="${camera_name}_mount_base_link"/>
+            <child link="${camera_name}_mount_point_1"/>
+            <origin xyz="0.17975 0.05775 0" rpy="0 0 0" />
+        </joint>
+        <joint name="${camera_name}_mount_point_2_joint" type="fixed">
+            <parent link="${camera_name}_mount_base_link"/>
+            <child link="${camera_name}_mount_point_2"/>
+            <origin xyz="-0.17975 0.05775 0" rpy="0 0 0" />
+        </joint>
+        <joint name="${camera_name}_mount_point_3_joint" type="fixed">
+            <parent link="${camera_name}_mount_base_link"/>
+            <child link="${camera_name}_mount_point_3"/>
+            <origin xyz="0.17975 -0.05775 0" rpy="0 0 0" />
+        </joint>
+        <joint name="${camera_name}_mount_point_4_joint" type="fixed">
+            <parent link="${camera_name}_mount_base_link"/>
+            <child link="${camera_name}_mount_point_4"/>
+            <origin xyz="-0.17975 -0.05775 0" rpy="0 0 0" />
+        </joint>
     </xacro:macro>
 </robot>
